Commit message: Update Indy Wuji reach environment

File: nrmk_isaaclab_wuji/isaac_neuromeka/assets/model/urdf/wuji_right/wuji_right.urdf (robot description, URDF)
Before this commit: robot wujihand-right-v1.0.2, 26 links, 25 joints
Links:
- link finger1_link1: geometry collision mesh filename=meshes/finger1_link1_collision.STL; visual mesh filename=meshes/finger1_link1.STL
- link finger1_link2: geometry collision mesh filename=meshes/finger1_link2_collision.STL; visual mesh filename=meshes/finger1_link2.STL
- link finger1_link3: geometry collision mesh filename=meshes/finger1_link3_collision.STL; visual mesh filename=meshes/finger1_link3.STL
- link finger1_link4: geometry collision mesh filename=meshes/finger1_link4_collision.STL; visual mesh filename=meshes/finger1_link4.STL
- link finger2_link1: geometry collision mesh filename=meshes/finger2_link1_collision.STL; visual mesh filename=meshes/finger2_link1.STL
- link finger2_link2: geometry collision mesh filename=meshes/finger2_link2_collision.STL; visual mesh filename=meshes/finger2_link2.STL
- link finger2_link3: geometry collision mesh filename=meshes/finger2_link3_collision.STL; visual mesh filename=meshes/finger2_link3.STL
- link finger2_link4: geometry collision mesh filename=meshes/finger2_link4_collision.STL; visual mesh filename=meshes/finger2_link4.STL
- link finger3_link1: geometry collision mesh filename=meshes/finger3_link1_collision.STL; visual mesh filename=meshes/finger3_link1.STL
- link finger3_link2: geometry collision mesh filename=meshes/finger3_link2_collision.STL; visual mesh filename=meshes/finger3_link2.STL
- link finger3_link3: geometry collision mesh filename=meshes/finger3_link3_collision.STL; visual mesh filename=meshes/finger3_link3.STL
- link finger3_link4: geometry collision mesh filename=meshes/finger3_link4_collision.STL; visual mesh filename=meshes/finger3_link4.STL
- link finger4_link1: geometry collision mesh filename=meshes/finger4_link1_collision.STL; visual mesh filename=meshes/finger4_link1.STL
- link finger4_link2: geometry collision mesh filename=meshes/finger4_link2_collision.STL; visual mesh filename=meshes/finger4_link2.STL
- link finger4_link3: geometry collision mesh filename=meshes/finger4_link3_collision.STL; visual mesh filename=meshes/finger4_link3.STL
- link finger4_link4: geometry collision mesh filename=meshes/finger4_link4_collision.STL; visual mesh filename=meshes/finger4_link4.STL
- link finger5_link1: geometry collision mesh filename=meshes/finger5_link1_collision.STL; visual mesh filename=meshes/finger5_link1.STL
- link finger5_link2: geometry collision mesh filename=meshes/finger5_link2_collision.STL; visual mesh filename=meshes/finger5_link2.STL
- link finger5_link3: geometry collision mesh filename=meshes/finger5_link3_collision.STL; visual mesh filename=meshes/finger5_link3.STL
- link finger5_link4: geometry collision mesh filename=meshes/finger5_link4_collision.STL; visual mesh filename=meshes/finger5_link4.STL
- link palm_link: geometry collision mesh filename=meshes/palm_link_collision.STL; visual mesh filename=meshes/palm_link.STL
